Commit message: Added Base_link

File: revolt_description/urdf/revolt.urdf.xacro (robot description, xacro)
@@ -1,499 +1,410 @@
 <?xml version="1.0"?>
 <robot xmlns:xacro="http://www.ros.org/wiki/xacro" name="revolt">
-    <!-- CHASSIS -->
-<link name="chassis">
-<visual>
-    <origin
-        xyz="0.0010000000000000427384 -1.3877787807814456755e-17 0.034499999999999975131"
-        rpy="3.141592653589793116 -0 1.5992498330910002766e-16" />
-    <geometry>
-        <mesh filename="file://$(find revolt_description)/meshes/mouth.stl" />
-    </geometry>
-    <material name="mouth_material">
-        <color
-            rgba="0.18431372549019608975 0.18431372549019608975 0.18039215686274509554 1.0" />
-    </material>
-</visual>
-<!-- <collision>
-    <origin
-        xyz="0.0010000000000000427384 -1.3877787807814456755e-17 0.034499999999999975131"
-        rpy="3.141592653589793116 -0 1.5992498330910002766e-16" />
-    <geometry>
-        <mesh filename="file://$(find revolt_description)/meshes/mouth.stl" />
-    </geometry>
-</collision> -->
-<visual>
-    <origin
-        xyz="0.0010000000000000572667 -2.0559984270640541126e-11 0.081246835314834925379"
-        rpy="3.877409121342316078e-26 2.0033280460268717061e-25 2.4319171015598684215e-16" />
-    <geometry>
-        <mesh filename="file://$(find revolt_description)/meshes/camera_deck.stl" />
-    </geometry>
-    <material name="camera_deck_material">
-        <color
-            rgba="0.91764705882352937127 0.91764705882352937127 0.91764705882352937127 1.0" />
-    </material>
-</visual>
-<!-- Shapes for camera_deck -->
-<collision>
-    <origin
-        xyz="0.0010005000000000577667 -2.0002055999002095288e-07 0.082746835314834926711"
-        rpy="-3.877409121342316078e-26 -2.0033280460268717061e-25 -3.141592653589793116" />
-    <geometry>
-        <box size="0.24927900000000000058 0.19929299999999999793 0.0030000000000000000625" />
-    </geometry>
-</collision>
-<visual>
-    <origin
-        xyz="-0.094939000879476515005 -2.5246608970075357092e-10 -0.0049999999999999983694"
-        rpy="-1.570796326794896558 -0 -1.570796326794896558" />
-    <geometry>
-        <mesh filename="file://$(find revolt_description)/meshes/caster_base_plate.stl" />
-    </geometry>
-    <material name="caster_base_plate_material">
-        <color
-            rgba="0.49803921568627451677 0.49803921568627451677 0.49803921568627451677 1.0" />
-    </material>
-</visual>
-<!-- <collision>
-    <origin
-        xyz="-0.094939000879476515005 -2.5246608970075357092e-10 -0.0049999999999999983694"
-        rpy="-1.570796326794896558 -0 -1.570796326794896558" />
-    <geometry>
-        <mesh filename="file://$(find revolt_description)/meshes/caster_base_plate.stl" />
-    </geometry>
-</collision> -->
-<visual>
-    <origin
-        xyz="0.00099999999998273778751 -0.00011057728351647477805 0.081207412577658427688"
-        rpy="2.1346669524422006952e-16 1.3293600162729647547e-12 1.3216940769347106485e-16" />
-    <geometry>
-        <mesh filename="file://$(find revolt_description)/meshes/camera_holder_cover.stl" />
-    </geometry>
-    <material name="camera_holder_cover_material">
-        <color
-            rgba="0.91764705882352937127 0.91764705882352937127 0.91764705882352937127 1.0" />
-    </material>
-</visual>
-<!-- <collision>
-    <origin
-        xyz="0.00099999999998273778751 -0.00011057728351647477805 0.081207412577658427688"
-        rpy="2.1346669524422006952e-16 1.3293600162729647547e-12 1.3216940769347106485e-16" />
-    <geometry>
-        <mesh filename="file://$(find revolt_description)/meshes/camera_holder_cover.stl" />
-    </geometry>
-</collision> -->
-<visual>
-    <origin
-        xyz="0.0010000000000000603025 -2.0559984270640541126e-11 0.081246835314834925379"
-        rpy="-8.2583008268328957817e-25 1.2527111174909710518e-26 1.3216940769347106485e-16" />
-    <geometry>
-        <mesh filename="file://$(find revolt_description)/meshes/lidar_mount_cover.stl" />
-    </geometry>
-    <material name="lidar_mount_cover_material">
-        <color
-            rgba="0.15686274509803921351 0.16078431372549020772 0.16078431372549020772 1.0" />
-    </material>
-</visual>
-<!-- <collision>
-    <origin
-        xyz="0.0010000000000000603025 -2.0559984270640541126e-11 0.081246835314834925379"
-        rpy="-8.2583008268328957817e-25 1.2527111174909710518e-26 1.3216940769347106485e-16" />
-    <geometry>
-        <mesh filename="file://$(find revolt_description)/meshes/lidar_mount_cover.stl" />
-    </geometry>
-</collision> -->
-<visual>
-    <origin
-        xyz="0.0010000000000000149828 -1.3877787807814456755e-17 0.034500000000000002887"
-        rpy="3.141592653589793116 -0 1.3216940769347106485e-16" />
-    <geometry>
-        <mesh filename="file://$(find revolt_description)/meshes/body.stl" />
-    </geometry>
-    <material name="body_material">
-        <color
-            rgba="0.18431372549019608975 0.18431372549019608975 0.18039215686274509554 1.0" />
-    </material>
-</visual>
-<!-- Shapes for body -->
-<collision>
-    <origin
-        xyz="0.0010000000000000149828 -1.3877787807814456755e-17 -0.014499999999999999001"
-        rpy="3.141592653589793116 -0 -3.141592653589793116" />
-    <geometry>
-        <box size="0.14212600000000000233 0.16452699999999997882 0.0020000000000000000416" />
-    </geometry>
-</collision>
-<collision>
-    <origin xyz="0.12449999999999962486 5.0000000000294362862e-07 0.034500000000000002887"
-        rpy="-1.570796326794896558 -0 -1.570796326794896558" />
-    <geometry>
-        <box size="0.20016100000000000558 0.10000000000000000555 0.0030000000000000000625" />
-    </geometry>
-</collision>
-<collision>
-    <origin xyz="-0.12249999999999959532 -5.0000000001682141643e-07 0.034500050000000004324"
-        rpy="-1.570796326794896558 -0 1.57079632679489678" />
-    <geometry>
-        <box size="0.2004070000000000018 0.099495299999999994855 0.0030000000000000000625" />
-    </geometry>
-</collision>
-<collision>
-    <origin xyz="0.00045135000000001278698 0.098999999999999685474 0.06378895000000001092"
-        rpy="-1.570796326794896558 -0 4.0769347106295352723e-22" />
-    <geometry>
-        <box size="0.083071299999999986818 0.040414099999999994473 0.0020000000000000000416" />
-    </geometry>
-</collision>
-<collision>
-    <origin xyz="-0.082699499999999717681 0.098999999999999685474 0.034500000000000002887"
-        rpy="-1.570796326794896558 -0 4.0769347106295352723e-22" />
-    <geometry>
-        <box size="0.082917000000000004589 0.099797799999999992071 0.0020000000000000000416" />
-    </geometry>
-</collision>
-<collision>
-    <origin xyz="0.083849049999999758498 0.098999999999999699352 0.034306300000000004846"
-        rpy="-1.570796326794896558 -0 4.0769347106295352723e-22" />
-    <geometry>
-        <box size="0.083871300000000009733 0.099612599999999995593 0.0020000000000000000416" />
-    </geometry>
-</collision>
-<collision>
-    <origin xyz="0.00045145000000001414466 -0.098999999999999713229 0.06378899999999999848"
-        rpy="-1.570796326794896558 -0 -3.141592653589793116" />
-    <geometry>
-        <box size="0.082840099999999999847 0.04037840000000000179 0.0020000000000000000416" />
-    </geometry>
-</collision>
-<collision>
-    <origin xyz="-0.082699099999999706179 -0.098999999999999727107 0.034500000000000002887"
-        rpy="-1.570796326794896558 -0 -3.141592653589793116" />
-    <geometry>
-        <box size="0.083039199999999993573 0.10000000000000000555 0.0020000000000000000416" />
-    </geometry>
-</collision>
-<collision>
-    <origin xyz="0.083849349999999753247 -0.098999999999999713229 0.034306300000000004846"
-        rpy="-1.570796326794896558 -0 -3.141592653589793116" />
-    <geometry>
-        <box size="0.083955299999999996596 0.099612599999999995593 0.0020000000000000000416" />
-    </geometry>
-</collision>
-<visual>
-    <origin
-        xyz="0.0010000000000000290774 -1.3877787807814456755e-17 0.034499999999999989009"
-        rpy="3.141592653589793116 -0 -6.9058515519838533453e-17" />
-    <geometry>
-        <mesh filename="file://$(find revolt_description)/meshes/face.stl" />
-    </geometry>
-    <material name="face_material">
-        <color
-            rgba="0.91764705882352937127 0.91764705882352937127 0.91764705882352937127 1.0" />
-    </material>
-</visual>
-<!-- <collision>
-    <origin
-        xyz="0.0010000000000000290774 -1.3877787807814456755e-17 0.034499999999999989009"
-        rpy="3.141592653589793116 -0 -6.9058515519838533453e-17" />
-    <geometry>
-        <mesh filename="file://$(find revolt_description)/meshes/face.stl" />
-    </geometry>
-</collision> -->
-<visual>
-    <origin xyz="-0.09903076211353280256 -0.0095000000205599927083 0.094246835314834992436"
-        rpy="1.57079632679489678 8.2036283484800396443e-22 2.4319171015598684215e-16" />
-    <geometry>
-        <mesh filename="file://$(find revolt_description)/meshes/3_mm_screw.stl" />
-    </geometry>
-    <material name="3_mm_screw_material">
-        <color
-            rgba="0.91764705882352937127 0.91764705882352937127 0.91764705882352937127 1.0" />
-    </material>
-</visual>
-<!-- <collision>
-    <origin xyz="-0.09903076211353280256 -0.0095000000205599927083 0.094246835314834992436"
-        rpy="1.57079632679489678 8.2036283484800396443e-22 2.4319171015598684215e-16" />
-    <geometry>
-        <mesh filename="file://$(find revolt_description)/meshes/3_mm_screw.stl" />
-    </geometry>
-</collision> -->
-<visual>
-    <origin xyz="-0.099030762113532844193 0.011199999979449953846 0.094246835314834992436"
-        rpy="1.57079632679489678 -3.8851905562594939282e-25 2.4319171015598684215e-16" />
-    <geometry>
-        <mesh filename="file://$(find revolt_description)/meshes/bolt.stl" />
-    </geometry>
-    <material name="bolt_material">
-        <color
-            rgba="0.85098039215686271941 0.7568627450980391913 0.87058823529411766273 1.0" />
-    </material>
-</visual>
-<!-- <collision>
-    <origin xyz="-0.099030762113532844193 0.011199999979449953846 0.094246835314834992436"
-        rpy="1.57079632679489678 -3.8851905562594939282e-25 2.4319171015598684215e-16" />
-    <geometry>
-        <mesh filename="file://$(find revolt_description)/meshes/bolt.stl" />
-    </geometry>
-</collision> -->
-<visual>
-    <origin
-        xyz="0.00099999999998277378302 -0.0001500000205599955061 0.081246835314701948416"
-        rpy="2.1346669524422006952e-16 1.3293600162729647547e-12 1.3216940769347106485e-16" />
-    <geometry>
-        <mesh filename="file://$(find revolt_description)/meshes/camera_mount_upper.stl" />
-    </geometry>
-    <material name="camera_mount_upper_material">
-        <color
-            rgba="0.91764705882352937127 0.91764705882352937127 0.91764705882352937127 1.0" />
-    </material>
-</visual>
-<!-- <collision>
-    <origin
-        xyz="0.00099999999998277378302 -0.0001500000205599955061 0.081246835314701948416"
-        rpy="2.1346669524422006952e-16 1.3293600162729647547e-12 1.3216940769347106485e-16" />
-    <geometry>
-        <mesh filename="file://$(find revolt_description)/meshes/camera_mount_upper.stl" />
-    </geometry>
-</collision> -->
-<visual>
-    <origin xyz="0.068999999999769093262 -2.0545637251490718116e-11 0.15974683531486091881"
-        rpy="-1.5707963267949949238 8.8439464137082285948e-14 -3.0990345367881952932" />
-    <geometry>
-        <mesh filename="file://$(find revolt_description)/meshes/lidar.stl" />
-    </geometry>
-    <material name="lidar_material">
-        <color
-            rgba="0.43921568627450979783 0.43921568627450979783 0.43921568627450979783 1.0" />
-    </material>
-</visual>
-<!-- <collision>
-    <origin xyz="0.068999999999769093262 -2.0545637251490718116e-11 0.15974683531486091881"
-        rpy="-1.5707963267949949238 8.8439464137082285948e-14 -3.0990345367881952932" />
-    <geometry>
-        <mesh filename="file://$(find revolt_description)/meshes/lidar.stl" />
-    </geometry>
-</collision> -->
-<visual>
-    <origin
-        xyz="0.097009446841797256078 -2.4932854392201164728e-10 -0.0049999999999999983694"
-        rpy="-1.570796326794896558 -0 -1.570796326794896558" />
-    <geometry>
-        <mesh filename="file://$(find revolt_description)/meshes/caster_base_plate.stl" />
-    </geometry>
-    <material name="caster_base_plate_material">
-        <color
-            rgba="0.49803921568627451677 0.49803921568627451677 0.49803921568627451677 1.0" />
-    </material>
-</visual>
-<!-- <collision>
-    <origin
-        xyz="0.097009446841797256078 -2.4932854392201164728e-10 -0.0049999999999999983694"
-        rpy="-1.570796326794896558 -0 -1.570796326794896558" />
-    <geometry>
-        <mesh filename="file://$(find revolt_description)/meshes/caster_base_plate.stl" />
-    </geometry>
-</collision> -->
-<visual>
-    <origin
-        xyz="0.00099999999998277942087 -0.0001500000205599955061 0.081246835314701948416"
-        rpy="2.1346669524422006952e-16 1.3293600162729647547e-12 1.3216940769347106485e-16" />
-    <geometry>
-        <mesh filename="file://$(find revolt_description)/meshes/lens.stl" />
-    </geometry>
-    <material name="lens_material">
-        <color rgba="0 0 0 1.0" />
-    </material>
-</visual>
-<!-- <collision>
-    <origin
-        xyz="0.00099999999998277942087 -0.0001500000205599955061 0.081246835314701948416"
-        rpy="2.1346669524422006952e-16 1.3293600162729647547e-12 1.3216940769347106485e-16" />
-    <geometry>
-        <mesh filename="file://$(find revolt_description)/meshes/lens.stl" />
-    </geometry>
-</collision> -->
-<inertial>
-    <origin
-        xyz="0.0035619083245137942231 -3.5819939158716627821e-06 0.028737618229734977066"
-        rpy="0 0 0" />
-    <mass value="1.37541365667756188" />
-    <inertia ixx="0.0074546494857456293073" ixy="9.3739832173881354348e-07"
-        ixz="-0.00024696587687848359314" iyy="0.0085957720605103291739"
-        iyz="9.872940559510540863e-07" izz="0.011229185530590277478" />
-</inertial>
-</link>
-        <!-- IMU -->
-<link name="imu">
-<inertial>
-    <origin xyz="0 0 0" rpy="0 0 0" />
-    <mass value="1e-9" />
-    <inertia ixx="0" ixy="0" ixz="0" iyy="0" iyz="0" izz="0" />
-</inertial>
-</link>
-<joint name="imu_frame" type="fixed">
-<origin xyz="0.003014671106491673136 -2.7204542826982439085e-05 0.084246835314834914166"
-    rpy="3.877409121342316078e-26 2.0033280460268717061e-25 2.4319171015598684215e-16" />
-<parent link="chassis" />
-<child link="imu" />
-<axis xyz="0 0 0" />
-</joint>
-        <!-- CAMERA -->
-<link name="camera">
-<inertial>
-    <origin xyz="0 0 0" rpy="0 0 0" />
-    <mass value="1e-9" />
-    <inertia ixx="0" ixy="0" ixz="0" iyy="0" iyz="0" izz="0" />
-</inertial>
-</link>
-<joint name="camera_frame" type="fixed">
-<origin xyz="-0.10553981779667316598 -0.00016122176437623829642 0.12324683531484359467"
-    rpy="1.3216940769347106485e-16 -1.5707963267935671769 0" />
-<parent link="chassis" />
-<child link="camera" />
-<axis xyz="0 0 0" />
-</joint>
-        <!-- LIDAR -->
-<link name="lidar">
-<inertial>
-    <origin xyz="0 0 0" rpy="0 0 0" />
-    <mass value="1e-9" />
-    <inertia ixx="0" ixy="0" ixz="0" iyy="0" iyz="0" izz="0" />
-</inertial>
-</link>
-<joint name="lidar_frame" type="fixed">
-<origin xyz="0.068995117891150689604 0.00011464698805746520449 0.15024683531486093813"
-    rpy="9.8371194238862312071e-14 -8.8439464137082285948e-14 0.042558116801597767331" />
-<parent link="chassis" />
-<child link="lidar" />
-<axis xyz="0 0 0" />
-</joint>
-        <!-- LEFT WHEEL -->
-<link name="left_wheel">
-<visual>
-    <origin xyz="-3.0364619563320692272e-19 -3.252606517456513302e-19 0"
-        rpy="1.570796326794896558 -6.0896070622529636293e-33 0" />
-    <geometry>
-        <mesh filename="file://$(find revolt_description)/meshes/wheel.stl" />
-    </geometry>
-    <material name="wheel_material">
-        <color
-            rgba="0.18431372549019608975 0.18431372549019608975 0.18039215686274509554 1.0" />
-    </material>
-</visual>
-<collision>
-    <origin xyz="-3.0364619563320692272e-19 -3.252606517456513302e-19 0"
-        rpy="1.570796326794896558 -6.0896070622529636293e-33 0" />
-    <geometry>
-        <mesh filename="file://$(find revolt_description)/meshes/wheel.stl" />
-    </geometry>
-</collision>
-<visual>
-    <origin xyz="-3.0364619563320692272e-19 -3.252606517456513302e-19 0"
-        rpy="-1.570796326794896558 1.9428902930940190154e-16 3.141592653589793116" />
-    <geometry>
-        <mesh filename="file://$(find revolt_description)/meshes/tire.stl" />
-    </geometry>
-    <material name="tire_material">
-        <color
-            rgba="0.91764705882352937127 0.91764705882352937127 0.91764705882352937127 1.0" />
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
Commit message: Fixed orientation of wheels

File: revolt_description/urdf/revolt.urdf.xacro (robot description, xacro)
@@ -283,5 +283,5 @@
         <visual>
             <origin xyz="-3.0364619563320692272e-19 -3.252606517456513302e-19 0"
-                rpy="1.570796326794896558 -6.0896070622529636293e-33 0" />
+                rpy="-1.570796326794896558 -6.0896070622529636293e-33 0" />
             <geometry>
                 <mesh filename="file://$(find revolt_description)/meshes/wheel.stl" />
@@ -294,5 +294,5 @@
         <collision>
             <origin xyz="-3.0364619563320692272e-19 -3.252606517456513302e-19 0"
-                rpy="1.570796326794896558 -6.0896070622529636293e-33 0" />
+                rpy="-1.570796326794896558 -6.0896070622529636293e-33 0" />
             <geometry>
                 <mesh filename="file://$(find revolt_description)/meshes/wheel.stl" />
@@ -301,5 +301,5 @@
         <visual>
             <origin xyz="-3.0364619563320692272e-19 -3.252606517456513302e-19 0"
-                rpy="-1.570796326794896558 1.9428902930940190154e-16 3.141592653589793116" />
+                rpy="1.570796326794896558 1.9428902930940190154e-16 3.141592653589793116" />
             <geometry>
                 <mesh filename="file://$(find revolt_description)/meshes/tire.stl" />
@@ -312,5 +312,5 @@
         <collision>
             <origin xyz="-3.0364619563320692272e-19 -3.252606517456513302e-19 0"
-                rpy="-1.570796326794896558 1.9428902930940190154e-16 3.141592653589793116" />
+                rpy="1.570796326794896558 1.9428902930940190154e-16 3.141592653589793116" />
             <geometry>
                 <mesh filename="file://$(find revolt_description)/meshes/tire.stl" />
@@ -327,7 +327,7 @@
         </inertial>
     </link>
-    <joint name="left_wheel" type="continuous">
+    <joint name="left_wheel_joint" type="continuous">
         <origin xyz="-2.5283525075024694638e-17 -0.094499999999999917399 5.2041704279304212832e-18"
-            rpy="-1.570796326794896558 -0 8.3597150366120441552e-17" />
+            rpy="1.570796326794896558 0 8.3597150366120441552e-17" />
         <parent link="chassis" />
         <child link="left_wheel" />
@@ -340,5 +340,5 @@
         <visual>
             <origin xyz="-3.0364619563319459676e-19 -3.252606517456513302e-19 0"
-                rpy="1.570796326794896558 2.3592239273284571554e-16 0" />
+                rpy="-1.570796326794896558 2.3592239273284571554e-16 0" />
             <geometry>
                 <mesh filename="file://$(find revolt_description)/meshes/tire.stl" />
@@ -351,5 +351,5 @@
         <collision>
             <origin xyz="-3.0364619563319459676e-19 -3.252606517456513302e-19 0"
-                rpy="1.570796326794896558 2.3592239273284571554e-16 0" />
+                rpy="-1.570796326794896558 2.3592239273284571554e-16 0" />
             <geometry>
                 <mesh filename="file://$(find revolt_description)/meshes/tire.stl" />
@@ -358,5 +358,5 @@
         <visual>
             <origin xyz="-3.0364619563319459676e-19 -3.252606517456513302e-19 0"
-                rpy="1.570796326794896558 5.5760257437813084088e-33 0" />
+                rpy="-1.570796326794896558 5.5760257437813084088e-33 0" />
             <geometry>
                 <mesh filename="file://$(find revolt_description)/meshes/wheel.stl" />
@@ -369,5 +369,5 @@
         <collision>
             <origin xyz="-3.0364619563319459676e-19 -3.252606517456513302e-19 0"
-                rpy="1.570796326794896558 5.5760257437813084088e-33 0" />
+                rpy="-1.570796326794896558 5.5760257437813084088e-33 0" />
             <geometry>
                 <mesh filename="file://$(find revolt_description)/meshes/wheel.stl" />
@@ -384,10 +384,10 @@
         </inertial>
     </link>
-    <joint name="right_wheel" type="continuous">
+    <joint name="right_wheel_joint" type="continuous">
         <origin xyz="-5.9717925247838849906e-17 0.094499999999999431677 5.2041704279304212832e-18"
-            rpy="-1.570796326794896558 -0 3.141592653589793116" />
+            rpy="1.570796326794896558 -0 3.141592653589793116" />
         <parent link="chassis" />
         <child link="right_wheel" />
-        <axis xyz="0 0 1" />
+        <axis xyz="0 0 -1" />
         <limit effort="1" velocity="20" />
         <joint_properties friction="0.0" />
@@ -406,11 +406,4 @@
             </material>
         </visual>
-        <!-- <collision>
-    <origin xyz="0.013499999999999998113 2.2538635793787358001e-18 -0.017000000000000001221"
-        rpy="1.570796326794896336 -0 -2.8513139455734266103e-43" />
-    <geometry>
-        <mesh filename="file://$(find revolt_description)/meshes/caster_punch_bracket.stl" />
-    </geometry>
-</collision> -->
         <inertial>
             <origin xyz="0.006241639410146364135 0.00015992521741832878106 -0.008867539427835038901"
@@ -481,11 +474,4 @@
             </material>
         </visual>
-        <!-- <collision>
-    <origin xyz="0.013499999999999998113 2.2538635793787358001e-18 -0.017000000000000001221"
-        rpy="1.570796326794896336 -0 -1.1046173050810472067e-44" />
-    <geometry>
-        <mesh filename="file://$(find revolt_description)/meshes/caster_punch_bracket.stl" />
-    </geometry>
-</collision> -->
         <inertial>
             <origin xyz="0.006241639410146364135 0.00015992521741832878106 -0.008867539427835038901"
