Commit message: Added materials for urdf

File: revolt_description/urdf/revolt.urdf.xacro (robot description, xacro)
@@ -1,12 +1,15 @@
 <?xml version="1.0"?>
 <robot xmlns:xacro="http://www.ros.org/wiki/xacro" name="revolt">
+    <xacro:property name="package_name" value="revolt_description" />
+    <xacro:property name="robot_name" value="revolt" />
+    <xacro:include filename="$(find ${package_name})/urdf/include/materials.urdf.xacro" />
     <!-- ................................ BASE LINK .................................. -->
-    <link name="base_footprint"/>
-    <link name="base_link"/>
-        <joint name="base_joint" type="fixed">
-            <parent link="base_footprint" />
-            <child link="base_link" />
-            <origin xyz="0 0 0.0379" rpy="0 0 0" />
-        </joint>
+    <link name="base_footprint" />
+    <link name="base_link" />
+    <joint name="base_joint" type="fixed">
+        <parent link="base_footprint" />
+        <child link="base_link" />
+        <origin xyz="0 0 0.0379" rpy="0 0 0" />
+    </joint>
     <!-- ................................ CHASSIS .................................. -->
     <link name="chassis">
@@ -18,8 +21,5 @@
                 <mesh filename="file://$(find revolt_description)/meshes/mouth.stl" />
             </geometry>
-            <material name="mouth_material">
-                <color
-                    rgba="0.18431372549019608975 0.18431372549019608975 0.18039215686274509554 1.0" />
-            </material>
+            <material name="black" />
         </visual>
         <visual>
@@ -30,8 +30,5 @@
                 <mesh filename="file://$(find revolt_description)/meshes/camera_deck.stl" />
             </geometry>
-            <material name="camera_deck_material">
-                <color
-                    rgba="0.91764705882352937127 0.91764705882352937127 0.91764705882352937127 1.0" />
-            </material>
+            <material name="white" />
         </visual>
         <!-- Shapes for camera_deck -->
@@ -51,8 +48,5 @@
                 <mesh filename="file://$(find revolt_description)/meshes/caster_base_plate.stl" />
             </geometry>
-            <material name="caster_base_plate_material">
-                <color
-                    rgba="0.49803921568627451677 0.49803921568627451677 0.49803921568627451677 1.0" />
-            </material>
+            <material name="black" />
         </visual>
         <visual>
@@ -63,8 +57,5 @@
                 <mesh filename="file://$(find revolt_description)/meshes/camera_holder_cover.stl" />
             </geometry>
-            <material name="camera_holder_cover_material">
-                <color
-                    rgba="0.91764705882352937127 0.91764705882352937127 0.91764705882352937127 1.0" />
-            </material>
+            <material name="white" />
         </visual>
         <visual>
@@ -75,8 +66,5 @@
                 <mesh filename="file://$(find revolt_description)/meshes/lidar_mount_cover.stl" />
             </geometry>
-            <material name="lidar_mount_cover_material">
-                <color
-                    rgba="0.15686274509803921351 0.16078431372549020772 0.16078431372549020772 1.0" />
-            </material>
+            <material name="black" />
         </visual>
         <visual>
@@ -87,8 +75,5 @@
                 <mesh filename="file://$(find revolt_description)/meshes/body.stl" />
             </geometry>
-            <material name="body_material">
-                <color
-                    rgba="0.18431372549019608975 0.18431372549019608975 0.18039215686274509554 1.0" />
-            </material>
+            <material name="black" />
         </visual>
         <!-- Shapes for body -->
@@ -164,8 +149,5 @@
                 <mesh filename="file://$(find revolt_description)/meshes/face.stl" />
             </geometry>
-            <material name="face_material">
-                <color
-                    rgba="0.91764705882352937127 0.91764705882352937127 0.91764705882352937127 1.0" />
-            </material>
+            <material name="white" />
         </visual>
         <visual>
@@ -175,8 +157,5 @@
                 <mesh filename="file://$(find revolt_description)/meshes/3_mm_screw.stl" />
             </geometry>
-            <material name="3_mm_screw_material">
-                <color
-                    rgba="0.91764705882352937127 0.91764705882352937127 0.91764705882352937127 1.0" />
-            </material>
+            <material name="silver" />
         </visual>
         <visual>
@@ -186,8 +165,5 @@
                 <mesh filename="file://$(find revolt_description)/meshes/bolt.stl" />
             </geometry>
-            <material name="bolt_material">
-                <color
-                    rgba="0.85098039215686271941 0.7568627450980391913 0.87058823529411766273 1.0" />
-            </material>
+            <material name="silver" />
         </visual>
         <visual>
@@ -198,8 +174,5 @@
                 <mesh filename="file://$(find revolt_description)/meshes/camera_mount_upper.stl" />
             </geometry>
-            <material name="camera_mount_upper_material">
-                <color
-                    rgba="0.91764705882352937127 0.91764705882352937127 0.91764705882352937127 1.0" />
-            </material>
+            <material name="white" />
         </visual>
         <visual>
@@ -209,8 +182,5 @@
                 <mesh filename="file://$(find revolt_description)/meshes/lidar.stl" />
             </geometry>
-            <material name="lidar_material">
-                <color
-                    rgba="0.43921568627450979783 0.43921568627450979783 0.43921568627450979783 1.0" />
-            </material>
+            <material name="dark_grey" />
         </visual>
         <visual>
@@ -221,8 +191,5 @@
                 <mesh filename="file://$(find revolt_description)/meshes/caster_base_plate.stl" />
             </geometry>
-            <material name="caster_base_plate_material">
-                <color
-                    rgba="0.49803921568627451677 0.49803921568627451677 0.49803921568627451677 1.0" />
-            </material>
+            <material name="black" />
         </visual>
         <visual>
@@ -233,7 +200,5 @@
                 <mesh filename="file://$(find revolt_description)/meshes/lens.stl" />
             </geometry>
-            <material name="lens_material">
-                <color rgba="0 0 0 1.0" />
-            </material>
+            <material name="red" />
         </visual>
         <inertial>
@@ -253,5 +218,5 @@
     </joint>
     <!-- ................................ IMU .................................. -->
-    <link name="imu"/>
+    <link name="imu" />
     <joint name="imu_frame" type="fixed">
         <origin xyz="0.003014671106491673136 -2.7204542826982439085e-05 0.084246835314834914166"
@@ -262,5 +227,5 @@
     </joint>
     <!-- ................................ CAMERA .................................. -->
-    <link name="camera"/>
+    <link name="camera" />
     <joint name="camera_frame" type="fixed">
         <origin xyz="-0.10553981779667316598 -0.00016122176437623829642 0.12324683531484359467"
@@ -271,5 +236,5 @@
     </joint>
     <!-- ................................ LIDAR .................................. -->
-    <link name="lidar"/>
+    <link name="lidar" />
     <joint name="lidar_frame" type="fixed">
         <origin xyz="0.068995117891150689604 0.00011464698805746520449 0.15024683531486093813"
@@ -287,8 +252,5 @@
                 <mesh filename="file://$(find revolt_description)/meshes/wheel.stl" />
             </geometry>
-            <material name="wheel_material">
-                <color
-                    rgba="0.18431372549019608975 0.18431372549019608975 0.18039215686274509554 1.0" />
-            </material>
+            <material name="black" />
         </visual>
         <collision>
@@ -305,8 +267,5 @@
                 <mesh filename="file://$(find revolt_description)/meshes/tire.stl" />
             </geometry>
-            <material name="tire_material">
-                <color
-                    rgba="0.91764705882352937127 0.91764705882352937127 0.91764705882352937127 1.0" />
-            </material>
+            <material name="white" />
         </visual>
         <collision>
@@ -344,8 +303,5 @@
                 <mesh filename="file://$(find revolt_description)/meshes/tire.stl" />
             </geometry>
-            <material name="tire_material">
-                <color
-                    rgba="0.91764705882352937127 0.91764705882352937127 0.91764705882352937127 1.0" />
-            </material>
+            <material name="white" />
         </visual>
         <collision>
@@ -362,8 +318,5 @@
                 <mesh filename="file://$(find revolt_description)/meshes/wheel.stl" />
             </geometry>
-            <material name="wheel_material">
-                <color
-                    rgba="0.18431372549019608975 0.18431372549019608975 0.18039215686274509554 1.0" />
-            </material>
+            <material name="black" />
         </visual>
         <collision>
@@ -393,5 +346,5 @@
         <joint_properties friction="0.0" />
     </joint>
-    <!-- ................................ CASTER WHEEL .................................. -->
+    <!-- ................................ FRONT CASTER WHEEL .................................. -->
     <link name="caster_punch_bracket">
         <visual>
@@ -401,8 +354,5 @@
                 <mesh filename="file://$(find revolt_description)/meshes/caster_punch_bracket.stl" />
             </geometry>
-            <material name="caster_punch_bracket_material">
-                <color
-                    rgba="0.91764705882352937127 0.91764705882352937127 0.91764705882352937127 1.0" />
-            </material>
+            <material name="silver" />
         </visual>
         <inertial>
@@ -422,8 +372,5 @@
                 <mesh filename="file://$(find revolt_description)/meshes/caster_wheel.stl" />
             </geometry>
-            <material name="caster_wheel_material">
-                <color
-                    rgba="0.49803921568627451677 0.49803921568627451677 0.49803921568627451677 1.0" />
-            </material>
+            <material name="black" />
         </visual>
         <collision>
@@ -462,4 +409,5 @@
         <joint_properties friction="0.0" />
     </joint>
+    <!-- ................................ BACK CASTER WHEEL .................................. -->
     <link name="caster_punch_bracket_2">
         <visual>
@@ -469,8 +417,5 @@
                 <mesh filename="file://$(find revolt_description)/meshes/caster_punch_bracket.stl" />
             </geometry>
-            <material name="caster_punch_bracket_material">
-                <color
-                    rgba="0.91764705882352937127 0.91764705882352937127 0.91764705882352937127 1.0" />
-            </material>
+            <material name="silver" />
         </visual>
         <inertial>
@@ -490,8 +435,5 @@
                 <mesh filename="file://$(find revolt_description)/meshes/caster_wheel.stl" />
             </geometry>
-            <material name="caster_wheel_material">
-                <color
-                    rgba="0.49803921568627451677 0.49803921568627451677 0.49803921568627451677 1.0" />
-            </material>
+            <material name="black" />
         </visual>
         <collision>

Commit message: Fixed meshes

File: revolt_description/urdf/revolt.urdf.xacro (robot description, xacro)
@@ -1,7 +1,32 @@
 <?xml version="1.0"?>
 <robot xmlns:xacro="http://www.ros.org/wiki/xacro" name="revolt">
-    <xacro:property name="package_name" value="revolt_description" />
-    <xacro:property name="robot_name" value="revolt" />
-    <xacro:include filename="$(find ${package_name})/urdf/include/materials.urdf.xacro" />
+    <!-- <xacro:property name="package_name" value="revolt_description" />
+    <xacro:property name="robot_name" value="revolt" /> -->
+    <!-- <xacro:include filename="$(find ${package_name})/urdf/include/materials.urdf.xacro" /> -->
+        <!-- RVIZ material RGBA definition. -->
+  <material name="yellow">
+    <color rgba="1 0.95 0 1"/>
+  </material>
+  <material name="blue">
+    <color rgba="0 0 1 1"/>
+  </material>
+  <material name="light_blue">
+    <color rgba="0 0.5 0.8 1"/>
+  </material>
+  <material name="black">
+    <color rgba="0 0 0 1"/>
+  </material>
+  <material name="white">
+    <color rgba="1 1 1 1"/>
+  </material>
+  <material name="red">
+    <color rgba="0.8 0.0 0.0 1.0"/>
+  </material>
+  <material name="silver">
+    <color rgba="0.79 0.82 0.93 1"/>
+  </material>
+  <material name="dark_grey">
+    <color rgba="0.3 0.3 0.3 1"/>
+  </material>
     <!-- ................................ BASE LINK .................................. -->
     <link name="base_footprint" />
@@ -19,5 +44,5 @@
                 rpy="3.141592653589793116 -0 1.5992498330910002766e-16" />
             <geometry>
-                <mesh filename="file://$(find revolt_description)/meshes/mouth.stl" />
+                <mesh filename="package://revolt_description/meshes/mouth.dae" />
             </geometry>
             <material name="black" />
@@ -28,5 +53,5 @@
                 rpy="3.877409121342316078e-26 2.0033280460268717061e-25 2.4319171015598684215e-16" />
             <geometry>
-                <mesh filename="file://$(find revolt_description)/meshes/camera_deck.stl" />
+                <mesh filename="package://revolt_description/meshes/camera_deck.dae" />
             </geometry>
             <material name="white" />
@@ -46,5 +71,5 @@
                 rpy="-1.570796326794896558 -0 -1.570796326794896558" />
             <geometry>
-                <mesh filename="file://$(find revolt_description)/meshes/caster_base_plate.stl" />
+                <mesh filename="package://revolt_description/meshes/caster_base_plate.dae" />
             </geometry>
             <material name="black" />
@@ -55,5 +80,5 @@
                 rpy="2.1346669524422006952e-16 1.3293600162729647547e-12 1.3216940769347106485e-16" />
             <geometry>
-                <mesh filename="file://$(find revolt_description)/meshes/camera_holder_cover.stl" />
+                <mesh filename="package://revolt_description/meshes/camera_holder_cover.dae" />
             </geometry>
             <material name="white" />
@@ -64,5 +89,5 @@
                 rpy="-8.2583008268328957817e-25 1.2527111174909710518e-26 1.3216940769347106485e-16" />
             <geometry>
-                <mesh filename="file://$(find revolt_description)/meshes/lidar_mount_cover.stl" />
+                <mesh filename="package://revolt_description/meshes/lidar_mount_cover.dae" />
             </geometry>
             <material name="black" />
@@ -73,7 +98,6 @@
                 rpy="3.141592653589793116 -0 1.3216940769347106485e-16" />
             <geometry>
-                <mesh filename="file://$(find revolt_description)/meshes/body.stl" />
-            </geometry>
-            <material name="black" />
+                <mesh filename="package://revolt_description/meshes/body.dae" />
+            </geometry>
         </visual>
         <!-- Shapes for body -->
@@ -147,5 +171,5 @@
                 rpy="3.141592653589793116 -0 -6.9058515519838533453e-17" />
             <geometry>
-                <mesh filename="file://$(find revolt_description)/meshes/face.stl" />
+                <mesh filename="package://revolt_description/meshes/face.dae" />
             </geometry>
             <material name="white" />
@@ -155,5 +179,5 @@
                 rpy="1.57079632679489678 8.2036283484800396443e-22 2.4319171015598684215e-16" />
             <geometry>
-                <mesh filename="file://$(find revolt_description)/meshes/3_mm_screw.stl" />
+                <mesh filename="package://revolt_description/meshes/screw.dae" />
             </geometry>
             <material name="silver" />
@@ -163,5 +187,5 @@
                 rpy="1.57079632679489678 -3.8851905562594939282e-25 2.4319171015598684215e-16" />
             <geometry>
-                <mesh filename="file://$(find revolt_description)/meshes/bolt.stl" />
+                <mesh filename="package://revolt_description/meshes/bolt.dae" />
             </geometry>
             <material name="silver" />
@@ -172,5 +196,5 @@
                 rpy="2.1346669524422006952e-16 1.3293600162729647547e-12 1.3216940769347106485e-16" />
             <geometry>
-                <mesh filename="file://$(find revolt_description)/meshes/camera_mount_upper.stl" />
+                <mesh filename="package://revolt_description/meshes/camera_mount_upper.dae" />
             </geometry>
             <material name="white" />
@@ -180,5 +204,5 @@
                 rpy="-1.5707963267949949238 8.8439464137082285948e-14 -3.0990345367881952932" />
             <geometry>
-                <mesh filename="file://$(find revolt_description)/meshes/lidar.stl" />
+                <mesh filename="package://revolt_description/meshes/lidar.dae" />
             </geometry>
             <material name="dark_grey" />
@@ -189,7 +213,7 @@
                 rpy="-1.570796326794896558 -0 -1.570796326794896558" />
             <geometry>
-                <mesh filename="file://$(find revolt_description)/meshes/caster_base_plate.stl" />
-            </geometry>
-            <material name="black" />
+                <mesh filename="package://revolt_description/meshes/caster_base_plate.dae" />
+            </geometry>
+            <material name="black"/>
         </visual>
         <visual>
@@ -198,7 +222,7 @@
                 rpy="2.1346669524422006952e-16 1.3293600162729647547e-12 1.3216940769347106485e-16" />
             <geometry>
-                <mesh filename="file://$(find revolt_description)/meshes/lens.stl" />
-            </geometry>
-            <material name="red" />
+                <mesh filename="package://revolt_description/meshes/lens.dae" />
+            </geometry>
+            <material name="red"/>
         </visual>
         <inertial>
@@ -250,5 +274,5 @@
                 rpy="-1.570796326794896558 -6.0896070622529636293e-33 0" />
             <geometry>
-                <mesh filename="file://$(find revolt_description)/meshes/wheel.stl" />
+                <mesh filename="package://revolt_description/meshes/wheel.dae" />
             </geometry>
             <material name="black" />
@@ -258,5 +282,5 @@
                 rpy="-1.570796326794896558 -6.0896070622529636293e-33 0" />
             <geometry>
-                <mesh filename="file://$(find revolt_description)/meshes/wheel.stl" />
+                <mesh filename="package://revolt_description/meshes/wheel.dae" />
             </geometry>
         </collision>
@@ -265,5 +289,5 @@
                 rpy="1.570796326794896558 1.9428902930940190154e-16 3.141592653589793116" />
             <geometry>
-                <mesh filename="file://$(find revolt_description)/meshes/tire.stl" />
+                <mesh filename="package://revolt_description/meshes/tire.dae" />
             </geometry>
             <material name="white" />
@@ -273,5 +297,5 @@
                 rpy="1.570796326794896558 1.9428902930940190154e-16 3.141592653589793116" />
             <geometry>
-                <mesh filename="file://$(find revolt_description)/meshes/tire.stl" />
+                <mesh filename="package://revolt_description/meshes/tire.dae" />
             </geometry>
         </collision>
@@ -301,5 +325,5 @@
                 rpy="-1.570796326794896558 2.3592239273284571554e-16 0" />
             <geometry>
-                <mesh filename="file://$(find revolt_description)/meshes/tire.stl" />
+                <mesh filename="package://revolt_description/meshes/tire.dae" />
             </geometry>
             <material name="white" />
@@ -309,5 +333,5 @@
                 rpy="-1.570796326794896558 2.3592239273284571554e-16 0" />
             <geometry>
-                <mesh filename="file://$(find revolt_description)/meshes/tire.stl" />
+                <mesh filename="package://revolt_description/meshes/tire.dae" />
             </geometry>
         </collision>
@@ -316,5 +340,5 @@
                 rpy="-1.570796326794896558 5.5760257437813084088e-33 0" />
             <geometry>
-                <mesh filename="file://$(find revolt_description)/meshes/wheel.stl" />
+                <mesh filename="package://revolt_description/meshes/wheel.dae" />
             </geometry>
             <material name="black" />
@@ -324,5 +348,5 @@
                 rpy="-1.570796326794896558 5.5760257437813084088e-33 0" />
             <geometry>
-                <mesh filename="file://$(find revolt_description)/meshes/wheel.stl" />
+                <mesh filename="package://revolt_description/meshes/wheel.dae" />
             </geometry>
         </collision>
@@ -352,5 +376,5 @@
                 rpy="1.570796326794896336 -0 -2.8513139455734266103e-43" />
             <geometry>
-                <mesh filename="file://$(find revolt_description)/meshes/caster_punch_bracket.stl" />
+                <mesh filename="package://revolt_description/meshes/caster_punch_bracket.dae" />
             </geometry>
             <material name="silver" />
@@ -370,5 +394,5 @@
                 rpy="0 2.8513139455734266103e-43 3.9877083809531582924e-48" />
             <geometry>
-                <mesh filename="file://$(find revolt_description)/meshes/caster_wheel.stl" />
+                <mesh filename="package://revolt_description/meshes/caster_wheel.dae" />
             </geometry>
             <material name="black" />
@@ -378,5 +402,5 @@
                 rpy="0 2.8513139455734266103e-43 3.9877083809531582924e-48" />
             <geometry>
-                <mesh filename="file://$(find revolt_description)/meshes/caster_wheel.stl" />
+                <mesh filename="package://revolt_description/meshes/caster_wheel.dae" />
             </geometry>
         </collision>
@@ -415,5 +439,5 @@
                 rpy="1.570796326794896336 -0 -1.1046173050810472067e-44" />
             <geometry>
-                <mesh filename="file://$(find revolt_description)/meshes/caster_punch_bracket.stl" />
+                <mesh filename="package://revolt_description/meshes/caster_punch_bracket.dae" />
             </geometry>
             <material name="silver" />
@@ -433,5 +457,5 @@
                 rpy="0 -8.2173010960533594582e-33 -5.4231385880628728748e-48" />
             <geometry>
-                <mesh filename="file://$(find revolt_description)/meshes/caster_wheel.stl" />
+                <mesh filename="package://revolt_description/meshes/caster_wheel.dae" />
             </geometry>
             <material name="black" />
@@ -441,5 +465,5 @@
                 rpy="0 -8.2173010960533594582e-33 -5.4231385880628728748e-48" />
             <geometry>
-                <mesh filename="file://$(find revolt_description)/meshes/caster_wheel.stl" />
+                <mesh filename="package://revolt_description/meshes/caster_wheel.dae" />
             </geometry>
         </collision>
