Commit message: removed custom rviz materials

File: revolt_description/urdf/revolt.urdf.xacro (robot description, xacro)
@@ -1,32 +1,6 @@
 <?xml version="1.0"?>
 <robot xmlns:xacro="http://www.ros.org/wiki/xacro" name="revolt">
-    <!-- <xacro:property name="package_name" value="revolt_description" />
-    <xacro:property name="robot_name" value="revolt" /> -->
-    <!-- <xacro:include filename="$(find ${package_name})/urdf/include/materials.urdf.xacro" /> -->
-        <!-- RVIZ material RGBA definition. -->
-  <material name="yellow">
-    <color rgba="1 0.95 0 1"/>
-  </material>
-  <material name="blue">
-    <color rgba="0 0 1 1"/>
-  </material>
-  <material name="light_blue">
-    <color rgba="0 0.5 0.8 1"/>
-  </material>
-  <material name="black">
-    <color rgba="0 0 0 1"/>
-  </material>
-  <material name="white">
-    <color rgba="1 1 1 1"/>
-  </material>
-  <material name="red">
-    <color rgba="0.8 0.0 0.0 1.0"/>
-  </material>
-  <material name="silver">
-    <color rgba="0.79 0.82 0.93 1"/>
-  </material>
-  <material name="dark_grey">
-    <color rgba="0.3 0.3 0.3 1"/>
-  </material>
+    <xacro:property name="package_name" value="revolt_description" />
+    <xacro:property name="robot_name" value="revolt" />
     <!-- ................................ BASE LINK .................................. -->
     <link name="base_footprint" />
@@ -46,5 +20,4 @@
                 <mesh filename="package://revolt_description/meshes/mouth.dae" />
             </geometry>
-            <material name="black" />
         </visual>
         <visual>
@@ -55,5 +28,4 @@
                 <mesh filename="package://revolt_description/meshes/camera_deck.dae" />
             </geometry>
-            <material name="white" />
         </visual>
         <!-- Shapes for camera_deck -->
@@ -73,5 +45,4 @@
                 <mesh filename="package://revolt_description/meshes/caster_base_plate.dae" />
             </geometry>
-            <material name="black" />
         </visual>
         <visual>
@@ -82,5 +53,4 @@
                 <mesh filename="package://revolt_description/meshes/camera_holder_cover.dae" />
             </geometry>
-            <material name="white" />
         </visual>
         <visual>
@@ -91,5 +61,4 @@
                 <mesh filename="package://revolt_description/meshes/lidar_mount_cover.dae" />
             </geometry>
-            <material name="black" />
         </visual>
         <visual>
@@ -173,5 +142,4 @@
                 <mesh filename="package://revolt_description/meshes/face.dae" />
             </geometry>
-            <material name="white" />
         </visual>
         <visual>
@@ -181,5 +149,4 @@
                 <mesh filename="package://revolt_description/meshes/screw.dae" />
             </geometry>
-            <material name="silver" />
         </visual>
         <visual>
@@ -189,5 +156,4 @@
                 <mesh filename="package://revolt_description/meshes/bolt.dae" />
             </geometry>
-            <material name="silver" />
         </visual>
         <visual>
@@ -198,5 +164,4 @@
                 <mesh filename="package://revolt_description/meshes/camera_mount_upper.dae" />
             </geometry>
-            <material name="white" />
         </visual>
         <visual>
@@ -206,5 +171,4 @@
                 <mesh filename="package://revolt_description/meshes/lidar.dae" />
             </geometry>
-            <material name="dark_grey" />
         </visual>
         <visual>
@@ -215,5 +179,4 @@
                 <mesh filename="package://revolt_description/meshes/caster_base_plate.dae" />
             </geometry>
-            <material name="black"/>
         </visual>
         <visual>
@@ -224,5 +187,4 @@
                 <mesh filename="package://revolt_description/meshes/lens.dae" />
             </geometry>
-            <material name="red"/>
         </visual>
         <inertial>
@@ -276,5 +238,4 @@
                 <mesh filename="package://revolt_description/meshes/wheel.dae" />
             </geometry>
-            <material name="black" />
         </visual>
         <collision>
@@ -291,5 +252,4 @@
                 <mesh filename="package://revolt_description/meshes/tire.dae" />
             </geometry>
-            <material name="white" />
         </visual>
         <collision>
@@ -327,5 +287,4 @@
                 <mesh filename="package://revolt_description/meshes/tire.dae" />
             </geometry>
-            <material name="white" />
         </visual>
         <collision>
@@ -342,5 +301,4 @@
                 <mesh filename="package://revolt_description/meshes/wheel.dae" />
             </geometry>
-            <material name="black" />
         </visual>
         <collision>
@@ -378,5 +336,4 @@
                 <mesh filename="package://revolt_description/meshes/caster_punch_bracket.dae" />
             </geometry>
-            <material name="silver" />
         </visual>
         <inertial>
@@ -396,5 +353,4 @@
                 <mesh filename="package://revolt_description/meshes/caster_wheel.dae" />
             </geometry>
-            <material name="black" />
         </visual>
         <collision>
@@ -441,5 +397,4 @@
                 <mesh filename="package://revolt_description/meshes/caster_punch_bracket.dae" />
             </geometry>
-            <material name="silver" />
         </visual>
         <inertial>
@@ -459,5 +414,4 @@
                 <mesh filename="package://revolt_description/meshes/caster_wheel.dae" />
             </geometry>
-            <material name="black" />
         </visual>
         <collision>

Commit message: Gazebo spawner with diff drive plugin

File: revolt_description/urdf/revolt.urdf.xacro (robot description, xacro)
@@ -213,19 +213,19 @@
     </joint>
     <!-- ................................ CAMERA .................................. -->
-    <link name="camera" />
-    <joint name="camera_frame" type="fixed">
+    <link name="camera_link" />
+    <joint name="camera_joint" type="fixed">
         <origin xyz="-0.10553981779667316598 -0.00016122176437623829642 0.12324683531484359467"
             rpy="1.3216940769347106485e-16 -1.5707963267935671769 0" />
         <parent link="chassis" />
-        <child link="camera" />
+        <child link="camera_link" />
         <axis xyz="0 0 0" />
     </joint>
     <!-- ................................ LIDAR .................................. -->
-    <link name="lidar" />
-    <joint name="lidar_frame" type="fixed">
+    <link name="rplidar_laser_link" />
+    <joint name="rplidar_laser_joint" type="fixed">
         <origin xyz="0.068995117891150689604 0.00011464698805746520449 0.15024683531486093813"
             rpy="9.8371194238862312071e-14 -8.8439464137082285948e-14 0.042558116801597767331" />
         <parent link="chassis" />
-        <child link="lidar" />
+        <child link="rplidar_laser_link" />
         <axis xyz="0 0 0" />
     </joint>
@@ -371,5 +371,5 @@
         </inertial>
     </link>
-    <joint name="front_casterwheel" type="continuous">
+    <joint name="frontcaster_wheel_joint" type="continuous">
         <origin xyz="0.013500000000000025868 3.1212253173671393473e-18 -0.017000000000000001221"
             rpy="-1.570796326794896336 -0 3.141592653589793116" />
@@ -380,5 +380,5 @@
         <joint_properties friction="0.0" />
     </joint>
-    <joint name="frontcasterpuch" type="continuous">
+    <joint name="frontcaster_rotation_joint" type="continuous">
         <origin xyz="-0.094939000879477097872 -2.5246608566260299064e-10 -0.0080000000000000001665"
             rpy="0 -0 -3.141592653589793116" />
@@ -432,5 +432,5 @@
         </inertial>
     </link>
-    <joint name="back_casterwheel" type="continuous">
+    <joint name="backcaster_wheel_joint" type="continuous">
         <origin xyz="0.013499999999999998113 2.2538635793787358001e-18 -0.017000000000000001221"
             rpy="1.570796326794896336 -0 -3.4594555838018703633e-45" />
@@ -441,5 +441,5 @@
         <joint_properties friction="0.0" />
     </joint>
-    <joint name="backcasterpunch" type="continuous">
+    <joint name="backcaster_rotation_joint" type="continuous">
         <origin xyz="0.097009446841797339345 -2.4932854392201164728e-10 -0.0080000000000000001665"
             rpy="0 -0 1.3216940769347106485e-16" />

Commit message: Adjusted casterwheel

File: revolt_description/urdf/revolt.urdf.xacro (robot description, xacro)
@@ -381,5 +381,5 @@
     </joint>
     <joint name="frontcaster_rotation_joint" type="continuous">
-        <origin xyz="-0.094939000879477097872 -2.5246608566260299064e-10 -0.0080000000000000001665"
+        <origin xyz="-0.094939000879477097872 -2.5246608566260299064e-10 -0.0082499999999999969191"
             rpy="0 -0 -3.141592653589793116" />
         <parent link="chassis" />
@@ -442,5 +442,5 @@
     </joint>
     <joint name="backcaster_rotation_joint" type="continuous">
-        <origin xyz="0.097009446841797339345 -2.4932854392201164728e-10 -0.0080000000000000001665"
+        <origin xyz="0.097009446841797339345 -2.4932854392201164728e-10 -0.0082499999999999969191"
             rpy="0 -0 1.3216940769347106485e-16" />
         <parent link="chassis" />

Commit message: Optimized urdf

File: revolt_description/urdf/revolt.urdf.xacro (robot description, xacro)
@@ -15,19 +15,11 @@
         <visual>
             <origin
-                xyz="0.0010000000000000427384 -1.3877787807814456755e-17 0.034499999999999975131"
-                rpy="3.141592653589793116 -0 1.5992498330910002766e-16" />
-            <geometry>
-                <mesh filename="package://revolt_description/meshes/mouth.dae" />
-            </geometry>
-        </visual>
-        <visual>
-            <origin
-                xyz="0.0010000000000000572667 -2.0559984270640541126e-11 0.081246835314834925379"
-                rpy="3.877409121342316078e-26 2.0033280460268717061e-25 2.4319171015598684215e-16" />
-            <geometry>
-                <mesh filename="package://revolt_description/meshes/camera_deck.dae" />
-            </geometry>
-        </visual>
-        <!-- Shapes for camera_deck -->
+                xyz="0.0010000000000000149828 -1.3877787807814456755e-17 0.034500000000000002887"
+                rpy="3.141592653589793116 -0 1.3216940769347106485e-16" />
+            <geometry>
+                <mesh filename="package://revolt_description/meshes/revolt_chassis.dae" />
+            </geometry>
+        </visual>
+         <!-- simplified collisions -->
         <collision>
             <origin
@@ -38,37 +30,4 @@
             </geometry>
         </collision>
-        <visual>
-            <origin
-                xyz="-0.094939000879476515005 -2.5246608970075357092e-10 -0.0049999999999999983694"
-                rpy="-1.570796326794896558 -0 -1.570796326794896558" />
-            <geometry>
-                <mesh filename="package://revolt_description/meshes/caster_base_plate.dae" />
-            </geometry>
-        </visual>
-        <visual>
-            <origin
-                xyz="0.00099999999998273778751 -0.00011057728351647477805 0.081207412577658427688"
-                rpy="2.1346669524422006952e-16 1.3293600162729647547e-12 1.3216940769347106485e-16" />
-            <geometry>
-                <mesh filename="package://revolt_description/meshes/camera_holder_cover.dae" />
-            </geometry>
-        </visual>
-        <visual>
-            <origin
-                xyz="0.0010000000000000603025 -2.0559984270640541126e-11 0.081246835314834925379"
-                rpy="-8.2583008268328957817e-25 1.2527111174909710518e-26 1.3216940769347106485e-16" />
-            <geometry>
-                <mesh filename="package://revolt_description/meshes/lidar_mount_cover.dae" />
-            </geometry>
-        </visual>
-        <visual>
-            <origin
-                xyz="0.0010000000000000149828 -1.3877787807814456755e-17 0.034500000000000002887"
-                rpy="3.141592653589793116 -0 1.3216940769347106485e-16" />
-            <geometry>
-                <mesh filename="package://revolt_description/meshes/body.dae" />
-            </geometry>
-        </visual>
-        <!-- Shapes for body -->
         <collision>
             <origin
@@ -135,57 +94,4 @@
             </geometry>
         </collision>
-        <visual>
-            <origin
-                xyz="0.0010000000000000290774 -1.3877787807814456755e-17 0.034499999999999989009"
-                rpy="3.141592653589793116 -0 -6.9058515519838533453e-17" />
-            <geometry>
-                <mesh filename="package://revolt_description/meshes/face.dae" />
-            </geometry>
-        </visual>
-        <visual>
-            <origin xyz="-0.09903076211353280256 -0.0095000000205599927083 0.094246835314834992436"
-                rpy="1.57079632679489678 8.2036283484800396443e-22 2.4319171015598684215e-16" />
-            <geometry>
-                <mesh filename="package://revolt_description/meshes/screw.dae" />
-            </geometry>
-        </visual>
-        <visual>
-            <origin xyz="-0.099030762113532844193 0.011199999979449953846 0.094246835314834992436"
-                rpy="1.57079632679489678 -3.8851905562594939282e-25 2.4319171015598684215e-16" />
-            <geometry>
-                <mesh filename="package://revolt_description/meshes/bolt.dae" />
-            </geometry>
-        </visual>
-        <visual>
-            <origin
-                xyz="0.00099999999998277378302 -0.0001500000205599955061 0.081246835314701948416"
-                rpy="2.1346669524422006952e-16 1.3293600162729647547e-12 1.3216940769347106485e-16" />
-            <geometry>
-                <mesh filename="package://revolt_description/meshes/camera_mount_upper.dae" />
-            </geometry>
-        </visual>
-        <visual>
-            <origin xyz="0.068999999999769093262 -2.0545637251490718116e-11 0.15974683531486091881"
-                rpy="-1.5707963267949949238 8.8439464137082285948e-14 -3.0990345367881952932" />
-            <geometry>
-                <mesh filename="package://revolt_description/meshes/lidar.dae" />
-            </geometry>
-        </visual>
-        <visual>
-            <origin
-                xyz="0.097009446841797256078 -2.4932854392201164728e-10 -0.0049999999999999983694"
-                rpy="-1.570796326794896558 -0 -1.570796326794896558" />
-            <geometry>
-                <mesh filename="package://revolt_description/meshes/caster_base_plate.dae" />
-            </geometry>
-        </visual>
-        <visual>
-            <origin
-                xyz="0.00099999999998277942087 -0.0001500000205599955061 0.081246835314701948416"
-                rpy="2.1346669524422006952e-16 1.3293600162729647547e-12 1.3216940769347106485e-16" />
-            <geometry>
-                <mesh filename="package://revolt_description/meshes/lens.dae" />
-            </geometry>
-        </visual>
         <inertial>
             <origin
@@ -236,5 +142,5 @@
                 rpy="-1.570796326794896558 -6.0896070622529636293e-33 0" />
             <geometry>
-                <mesh filename="package://revolt_description/meshes/wheel.dae" />
+                <mesh filename="package://revolt_description/meshes/left_wheel.dae" />
             </geometry>
         </visual>
@@ -243,19 +149,5 @@
                 rpy="-1.570796326794896558 -6.0896070622529636293e-33 0" />
             <geometry>
-                <mesh filename="package://revolt_description/meshes/wheel.dae" />
-            </geometry>
-        </collision>
-        <visual>
-            <origin xyz="-3.0364619563320692272e-19 -3.252606517456513302e-19 0"
-                rpy="1.570796326794896558 1.9428902930940190154e-16 3.141592653589793116" />
-            <geometry>
-                <mesh filename="package://revolt_description/meshes/tire.dae" />
-            </geometry>
-        </visual>
-        <collision>
-            <origin xyz="-3.0364619563320692272e-19 -3.252606517456513302e-19 0"
-                rpy="1.570796326794896558 1.9428902930940190154e-16 3.141592653589793116" />
-            <geometry>
-                <mesh filename="package://revolt_description/meshes/tire.dae" />
+                <mesh filename="package://revolt_description/meshes/left_wheel.dae" />
             </geometry>
         </collision>
@@ -283,28 +175,14 @@
         <visual>
             <origin xyz="-3.0364619563319459676e-19 -3.252606517456513302e-19 0"
-                rpy="-1.570796326794896558 2.3592239273284571554e-16 0" />
-            <geometry>
-                <mesh filename="package://revolt_description/meshes/tire.dae" />
-            </geometry>
-        </visual>
-        <collision>
-            <origin xyz="-3.0364619563319459676e-19 -3.252606517456513302e-19 0"
-                rpy="-1.570796326794896558 2.3592239273284571554e-16 0" />
-            <geometry>
-                <mesh filename="package://revolt_description/meshes/tire.dae" />
-            </geometry>
-        </collision>
-        <visual>
+                rpy="-1.570796326794896558 5.5760257437813084088e-33 0" />
+            <geometry>
+                <mesh filename="package://revolt_description/meshes/right_wheel.dae" />
+            </geometry>
+        </visual>
+        <collision>
             <origin xyz="-3.0364619563319459676e-19 -3.252606517456513302e-19 0"
                 rpy="-1.570796326794896558 5.5760257437813084088e-33 0" />
             <geometry>
-                <mesh filename="package://revolt_description/meshes/wheel.dae" />
-            </geometry>
-        </visual>
-        <collision>
-            <origin xyz="-3.0364619563319459676e-19 -3.252606517456513302e-19 0"
-                rpy="-1.570796326794896558 5.5760257437813084088e-33 0" />
-            <geometry>
-                <mesh filename="package://revolt_description/meshes/wheel.dae" />
+                <mesh filename="package://revolt_description/meshes/right_wheel.dae" />
             </geometry>
         </collision>
