Commit message: Included revolt_control xacro

File: revolt_description/urdf/revolt.urdf.xacro (robot description, xacro)
@@ -21,5 +21,5 @@
             </geometry>
         </visual>
-         <!-- simplified collisions -->
+        <!-- simplified collisions -->
         <collision>
             <origin
@@ -249,22 +249,46 @@
         </inertial>
     </link>
-    <joint name="frontcaster_wheel_joint" type="continuous">
-        <origin xyz="0.013500000000000025868 3.1212253173671393473e-18 -0.017000000000000001221"
-            rpy="-1.570796326794896336 -0 3.141592653589793116" />
-        <parent link="caster_punch_bracket" />
-        <child link="caster_wheel" />
-        <axis xyz="0 0 1" />
-        <limit effort="1" velocity="20" />
-        <joint_properties friction="0.0" />
-    </joint>
-    <joint name="frontcaster_rotation_joint" type="continuous">
-        <origin xyz="-0.094939000879477097872 -2.5246608566260299064e-10 -0.0082499999999999969191"
-            rpy="0 -0 -3.141592653589793116" />
-        <parent link="chassis" />
-        <child link="caster_punch_bracket" />
-        <axis xyz="0 0 1" />
-        <limit effort="1" velocity="20" />
-        <joint_properties friction="0.0" />
-    </joint>
+    <xacro:if value="$(arg use_real_ros_control)">
+        <joint name="frontcaster_wheel_joint" type="fixed">
+            <origin xyz="0.013500000000000025868 3.1212253173671393473e-18 -0.017000000000000001221"
+                rpy="-1.570796326794896336 -0 3.141592653589793116" />
+            <parent link="caster_punch_bracket" />
+            <child link="caster_wheel" />
+            <axis xyz="0 0 1" />
+            <limit effort="1" velocity="20" />
+            <joint_properties friction="0.0" />
+        </joint>
+        <joint name="frontcaster_rotation_joint" type="fixed">
+            <origin
+                xyz="-0.094939000879477097872 -2.5246608566260299064e-10 -0.0082499999999999969191"
+                rpy="0 -0 -3.141592653589793116" />
+            <parent link="chassis" />
+            <child link="caster_punch_bracket" />
+            <axis xyz="0 0 1" />
+            <limit effort="1" velocity="20" />
+            <joint_properties friction="0.0" />
+        </joint>
+    </xacro:if>
+    <xacro:unless value="$(arg use_real_ros_control)">
+        <joint name="frontcaster_wheel_joint" type="continuous">
+            <origin xyz="0.013500000000000025868 3.1212253173671393473e-18 -0.017000000000000001221"
+                rpy="-1.570796326794896336 -0 3.141592653589793116" />
+            <parent link="caster_punch_bracket" />
+            <child link="caster_wheel" />
+            <axis xyz="0 0 1" />
+            <limit effort="1" velocity="20" />
+            <joint_properties friction="0.0" />
+        </joint>
+        <joint name="frontcaster_rotation_joint" type="continuous">
+            <origin
+                xyz="-0.094939000879477097872 -2.5246608566260299064e-10 -0.0082499999999999969191"
+                rpy="0 -0 -3.141592653589793116" />
+            <parent link="chassis" />
+            <child link="caster_punch_bracket" />
+            <axis xyz="0 0 1" />
+            <limit effort="1" velocity="20" />
+            <joint_properties friction="0.0" />
+        </joint>
+    </xacro:unless>
     <!-- ................................ BACK CASTER WHEEL .................................. -->
     <link name="caster_punch_bracket_2">
@@ -310,21 +334,49 @@
         </inertial>
     </link>
-    <joint name="backcaster_wheel_joint" type="continuous">
-        <origin xyz="0.013499999999999998113 2.2538635793787358001e-18 -0.017000000000000001221"
-            rpy="1.570796326794896336 -0 -3.4594555838018703633e-45" />
-        <parent link="caster_punch_bracket_2" />
-        <child link="caster_wheel_2" />
-        <axis xyz="0 0 1" />
-        <limit effort="1" velocity="20" />
-        <joint_properties friction="0.0" />
-    </joint>
-    <joint name="backcaster_rotation_joint" type="continuous">
-        <origin xyz="0.097009446841797339345 -2.4932854392201164728e-10 -0.0082499999999999969191"
-            rpy="0 -0 1.3216940769347106485e-16" />
-        <parent link="chassis" />
-        <child link="caster_punch_bracket_2" />
-        <axis xyz="0 0 1" />
-        <limit effort="1" velocity="20" />
-        <joint_properties friction="0.0" />
-    </joint>
+    <xacro:if value="$(arg use_real_ros_control)">
+        <joint name="backcaster_wheel_joint" type="fixed">
+            <origin xyz="0.013499999999999998113 2.2538635793787358001e-18 -0.017000000000000001221"
+                rpy="1.570796326794896336 -0 -3.4594555838018703633e-45" />
+            <parent link="caster_punch_bracket_2" />
+            <child link="caster_wheel_2" />
+            <axis xyz="0 0 1" />
+            <limit effort="1" velocity="20" />
+            <joint_properties friction="0.0" />
+        </joint>
+        <joint name="backcaster_rotation_joint" type="fixed">
+            <origin
+                xyz="0.097009446841797339345 -2.4932854392201164728e-10 -0.0082499999999999969191"
+                rpy="0 -0 1.3216940769347106485e-16" />
+            <parent link="chassis" />
+            <child link="caster_punch_bracket_2" />
+            <axis xyz="0 0 1" />
+            <limit effort="1" velocity="20" />
+            <joint_properties friction="0.0" />
+        </joint>
+    </xacro:if>
+    <xacro:unless value="$(arg use_real_ros_control)">
+        <joint name="backcaster_wheel_joint" type="continuous">
+            <origin xyz="0.013499999999999998113 2.2538635793787358001e-18 -0.017000000000000001221"
+                rpy="1.570796326794896336 -0 -3.4594555838018703633e-45" />
+            <parent link="caster_punch_bracket_2" />
+            <child link="caster_wheel_2" />
+            <axis xyz="0 0 1" />
+            <limit effort="1" velocity="20" />
+            <joint_properties friction="0.0" />
+        </joint>
+        <joint name="backcaster_rotation_joint" type="continuous">
+            <origin
+                xyz="0.097009446841797339345 -2.4932854392201164728e-10 -0.0082499999999999969191"
+                rpy="0 -0 1.3216940769347106485e-16" />
+            <parent link="chassis" />
+            <child link="caster_punch_bracket_2" />
+            <axis xyz="0 0 1" />
+            <limit effort="1" velocity="20" />
+            <joint_properties friction="0.0" />
+        </joint>
+    </xacro:unless>
+    <!-- ros2_control -->
+    <xacro:if value="$(arg use_real_ros_control)">
+        <xacro:include filename="$(find ${package_name})/urdf/include/revolt_control.urdf.xacro" />
+    </xacro:if>
 </robot>

Commit message: Added adjustable camera mount & fixes

File: revolt_description/urdf/revolt.urdf.xacro (robot description, xacro)
@@ -3,4 +3,5 @@
     <xacro:property name="package_name" value="revolt_description" />
     <xacro:property name="robot_name" value="revolt" />
+    <xacro:arg name="use_real_ros_control" default="false" />
     <!-- ................................ BASE LINK .................................. -->
     <link name="base_footprint" />
@@ -119,9 +120,27 @@
     </joint>
     <!-- ................................ CAMERA .................................. -->
+    <link name="camera_mount">
+        <visual>
+            <origin xyz="0.10003076211353316427 -0.013039422737043504519 -3.9422737043501517344e-05"
+                rpy="-1.5707963267948970021 -2.1130201991908125724e-32 -9.9510893136977499032e-54" />
+            <geometry>
+                <mesh filename="package://revolt_description/meshes/camera_mount.dae" />
+            </geometry>
+        </visual>
+    </link>
+    <joint name="camera_mount" type="fixed">
+        <origin xyz="-0.099030762113532788682 -2.0560008597292656995e-11 0.094246835314834839781"
+            rpy="1.570796326794896558 -2.0033280460268570124e-25 2.4319171023353502458e-16" />
+        <parent link="chassis" />
+        <child link="camera_mount" />
+        <axis xyz="0 0 1" />
+        <limit effort="1" velocity="20" />
+        <joint_properties friction="0.0" />
+    </joint>
     <link name="camera_link" />
     <joint name="camera_joint" type="fixed">
-        <origin xyz="-0.10553981779667316598 -0.00016122176437623829642 0.12324683531484359467"
-            rpy="1.3216940769347106485e-16 -1.5707963267935671769 0" />
-        <parent link="chassis" />
+        <origin xyz="-0.0065090556831789159187 0.028999999999999984124 1.1221743816224209809e-05"
+            rpy="-1.570796326794896558 3.2526065174728515974e-16 1.570796326794896558" />
+        <parent link="camera_mount" />
         <child link="camera_link" />
         <axis xyz="0 0 0" />
